Commit message: Teleoperated the maze & save the map

File: ddr/urdf/ddr.xacro (robot description, xacro)
@@ -98,5 +98,5 @@
   <joint name="camera_joint" type="fixed">
     <axis xyz="0 1 0" />
-    <origin xyz=".25 0 0" rpy="0 0 0"/>
+    <origin xyz=".27 0 0" rpy="0 0 0"/>
     <parent link="link_chassis"/>
     <child link="camera"/>
